Commit message: second commit

File: imr_description/urdf/imr.xacro (robot description, xacro)
@@ -15,5 +15,5 @@
       <mesh filename="package://imr_description/meshes/base_link.stl" scale="0.001 0.001 0.001"/>
     </geometry>
-    <material name="silver"/>
+    <material name="metal-material"/>
   </visual>
   <collision>
@@ -35,5 +35,5 @@
       <mesh filename="package://imr_description/meshes/lidar_1.stl" scale="0.001 0.001 0.001"/>
     </geometry>
-    <material name="silver"/>
+    <material name="blue"/>
   </visual>
   <collision>
@@ -47,5 +47,5 @@
   <inertial>
     <origin xyz="-5.551115123125783e-17 0.0 -0.032390624999999916" rpy="0 0 0"/>
-    <mass value="1.4205025342471604"/>
+    <mass value="2.4205025342471604"/>
     <inertia ixx="0.000818" iyy="0.000818" izz="0.000599" ixy="-0.0" iyz="-0.0" ixz="0.0"/>
   </inertial>
@@ -67,5 +67,5 @@
   <inertial>
     <origin xyz="-1.1102230246251565e-16 0.0 -0.032390624999999916" rpy="0 0 0"/>
-    <mass value="1.4205025342471604"/>
+    <mass value="2.4205025342471604"/>
     <inertia ixx="0.000818" iyy="0.000818" izz="0.000599" ixy="0.0" iyz="-0.0" ixz="0.0"/>
   </inertial>

File: imr_description/urdf/materials.xacro (robot description, xacro)
@@ -1,6 +1,12 @@
 <?xml version="1.0" ?>
-<robot name="imr" xmlns:xacro="http://www.ros.org/wiki/xacro" >
+<robot name="mobot" xmlns:xacro="http://www.ros.org/wiki/xacro" >
 <material name="silver">
   <color rgba="0.700 0.700 0.700 1.000"/>
 </material>
+<material name="blue">
+  <color rgba="0.000 0.000 1.000 1.000"/>
+</material>
+<material name="metal-material">
+  <color rgba="0.760 0.450 0.275 1.000"/>
+</material>
 </robot>
